File: Circuits/KiCAD/semg/semg.kicad_pcb (KiCad board)
At the start: 4 copper layers, 25 x 40 mm, 43 parts, among them J1 Miscelaneous, J10 Conn_01x08_Pin, J13 Conn_02x08_Odd_Even, J2 SPI, J3 Miscelaneous, J4 SPI, J5 505006-0812, J6 505006-0812, J7 CS_SPI, J8 CS_SPI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

Commit message: Final 3D models, test GUI with exe
Routing:
- net GND: track 41.7 -> 44.3 mm
Changed lines of the file:
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@@
+	)
+	(segment
+		(start 65.4 40.13)
+		(end 65.4 42.75)
+		(width 0.2)
+		(layer "F.Cu")
+		(net 5)
 	)
 	(segment
